Commit message: update ee origin to move it to the tip of the arm

File: motion_specification_action/urdf/Kinova_1.urdf (robot description, URDF)
Before this commit: robot GEN3_URDF_V12, 10 links, 9 joints
Joints:
- joint EndEffector: origin xyz=0 0 -0.0615250000000001 rpy=3.14159265358979 1.09937075168372E-32 0 -> xyz=0 0 -0.068 rpy=3.14159265358979 1.09937075168372E-32 0
